File: hardware/4StringDriver/4StringDriver.brd (EAGLE design)
At the start: 101.7 x 71.1 mm, 33 parts, among them J1 RJ45, J10 GND (1), J11 GND (2), J12 GND (3), J13 GND (4), J14 DOUT (1), J15 DOUT (2), J16 DOUT (3), J17 DOUT (4), J2 5VEN-IN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

Commit message: Updated 4StringDriver to v1.0a.
Parts:
- R2: value (none) -> 200
Other:
- board text removed: "Illumicone 4StringDriver Rev. 1.0 5/2016"
Changed lines of the file:
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@@
 <vertex x="59.69" y="34.29"/>
 </polygon>
-<text x="58.674" y="52.959" size="1.9304" layer="16" rot="MR0">Illumicone
-4StringDriver
-Rev. 1.0
-5/2016</text>
+<polygon width="0.4064" layer="42">
+<vertex x="0" y="0"/>
+<vertex x="0" y="10.16"/>
+<vertex x="6.35" y="10.16"/>
+<vertex x="12.7" y="3.81"/>
+<vertex x="12.7" y="1.27"/>
+<vertex x="12.7" y="0"/>
+</polygon>
+<polygon width="0.4064" layer="42">
+<vertex x="91.44" y="0"/>
+<vertex x="91.44" y="10.16"/>
+<vertex x="101.6" y="10.16"/>
+<vertex x="101.6" y="0"/>
+</polygon>
 </plain>
 <attributes>
@@
 </element>
 <element name="R1" library="rcl" package="0204/7" value="10k" x="15.24" y="46.99"/>
-<element name="R2" library="rcl" package="0204/7" value="" x="62.103" y="66.675" rot="R180"/>
+<element name="R2" library="rcl" package="0204/7" value="200" x="62.103" y="66.675" rot="R180"/>
 <element name="R3" library="rcl" package="0204/7" value="4.75k" x="74.93" y="52.07" rot="R180"/>
 <element name="R4" library="rcl" package="0204/7" value="3.83k" x="74.93" y="48.26" rot="R180"/>
@@
 <vertex x="63.5" y="53.975"/>
 <vertex x="63.5" y="69.85"/>
-<vertex x="92.71" y="69.85"/>
-<vertex x="92.71" y="62.23"/>
-<vertex x="100.33" y="62.23"/>
+<vertex x="91.44" y="69.85"/>
+<vertex x="91.44" y="60.96"/>
+<vertex x="100.33" y="60.96"/>
 <vertex x="100.33" y="48.26"/>
 <vertex x="81.28" y="48.26"/>
@@
 <polygon width="0.4064" layer="16" isolate="0.6096">
 <vertex x="0" y="0"/>
-<vertex x="0" y="71.12"/>
-<vertex x="8.89" y="71.12"/>
-<vertex x="8.89" y="60.96"/>
+<vertex x="0" y="60.96"/>
 <vertex x="12.7" y="60.96"/>
 <vertex x="12.7" y="53.34"/>
@@
 <polygon width="0.4064" layer="16" isolate="0.6096">
 <vertex x="10.795" y="69.977"/>
-<vertex x="22.86" y="69.723"/>
-<vertex x="22.86" y="55.753"/>
+<vertex x="22.987" y="69.977"/>
+<vertex x="22.987" y="55.88"/>
 <vertex x="15.24" y="55.88"/>
-<vertex x="15.24" y="63.5"/>
+<vertex x="15.24" y="63.627"/>
 <vertex x="10.795" y="63.627"/>
 </polygon>
@@
 </board>
 </drawing>
-<compatibility>
-<note version="6.3" minversion="6.2.2" severity="warning">
-Since Version 6.2.2 text objects can contain more than one line,
-which will not be processed correctly with this version.
-</note>
-</compatibility>
 </eagle>
