File: hardware/4StringDriver/4StringDriver.sch (EAGLE design)
At the start: 33 parts, among them J1 RJ45, J10 GND (1), J11 GND (2), J12 GND (3), J13 GND (4), J14 DOUT (1), J15 DOUT (2), J16 DOUT (3), J17 DOUT (4), J2 5VEN-IN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

Commit message: Updated 4StringDriver to v1.0a.
Parts:
- R2: value (none) -> 200
Changed lines of the file:
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@@
 <attributes>
 <attribute name="DESIGNER" value="Ross"/>
-<attribute name="VERSION" value="1.0"/>
+<attribute name="VERSION" value="1.0a"/>
 </attributes>
 <variantdefs>
@@
 <part name="SUPPLY3" library="supply2" deviceset="GND" device=""/>
 <part name="R1" library="rcl" deviceset="R-US_" device="0204/7" value="10k"/>
-<part name="R2" library="rcl" deviceset="R-US_" device="0204/7"/>
+<part name="R2" library="rcl" deviceset="R-US_" device="0204/7" value="200"/>
 <part name="R3" library="rcl" deviceset="R-US_" device="0204/7" value="4.75k"/>
 <part name="R4" library="rcl" deviceset="R-US_" device="0204/7" value="3.83k"/>
